File: pcb/power_supply.kicad_sch (KiCad schematic)
At the start: 14 parts, among them J201 1333870, SW201 SW_Push, U201 RT9080-33GJ5, U202 TLV803EF29DBZR

Commit message: WIP: Stashing work to mess with vm
Parts:
- PS201: footprint Converter_ACDC:Converter_ACDC_HiLink_HLK-PMxx -> ACDCLibrary:Converter_ACDC_HiLink_HLK-PMxx
Other:
- note added: "Decoupling cap needed?"
Changed lines of the file:
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@@
+		)
+	)
+	(text "Decoupling cap needed?\n"
+		(exclude_from_sim no)
+		(at 169.926 47.498 0)
+		(effects
+			(font
+				(size 1.27 1.27)
+			)
 		)
 	)
@@
 			)
 		)
-		(property "Footprint" "Converter_ACDC:Converter_ACDC_HiLink_HLK-PMxx"
+		(property "Footprint" "ACDCLibrary:Converter_ACDC_HiLink_HLK-PMxx"
 			(at 116.84 74.93 0)
 			(effects
