File: pcb/rp2350_core.kicad_sch (KiCad schematic)
At the start: 25 parts, among them J302 Debug Socket, U301 RP2350A-QFN60, Y301 ABM8-272-T3

Commit message: WIP: Stashing work to mess with vm
Parts:
- D301: footprint (none) -> LED_SMD:LED_0805_2012Metric
- J302: footprint (none) -> Connector_JST:JST_XH_B3B-XH-AM_1x03_P2.50mm_Vertical
Connections:
- net MAX_SPI.RX: now also U301.42 (GPIO28_ADC2); no longer U301.16 (GPIO12)
- net MAX_SPI.SCK: now also U301.40 (GPIO26_ADC0); no longer U301.17 (GPIO13)
Other:
- sheet Flash PSRAM ports: added QSPI{SD[0..3] SCLK CSN[0..1]}; removed none
- sheet Input Output ports: added BTN{0..2} SCREEN{SDA SCL} SPK; removed none
- sheet SD Card ports: added SDIO{SMD CLK D[0..3]} ~{SD_DET}; removed none
- sheet Temprature Control ports: added MAX_SPI{SCK[0..1] RX[0..1] ~{CS}[0..1]} SSR[0..1] FAN[0..1]; removed none
Changed lines of the file:
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@@
 	)
 	(bus_entry
+		(at 190.5 64.77)
+		(size -2.54 2.54)
+		(stroke
+			(width 0)
+			(type default)
+		)
+	)
+	(bus_entry
 		(at 73.66 86.36)
 		(size 2.54 -2.54)
@@
 	)
 	(bus_entry
+		(at 190.5 62.23)
+		(size -2.54 2.54)
+		(stroke
+			(width 0)
+			(type default)
+		)
+	)
+	(bus_entry
 		(at 73.66 92.71)
 		(size 2.54 -2.54)
@@
 	(wire
 		(pts
+			(xy 152.4 148.59) (xy 154.94 148.59)
+		)
+		(stroke
+			(width 0)
+			(type default)
+		)
+	)
+	(wire
+		(pts
 			(xy 152.4 85.09) (xy 154.94 85.09)
 		)
@@
 	(wire
 		(pts
-			(xy 175.26 59.69) (xy 187.96 59.69)
+			(xy 171.45 59.69) (xy 187.96 59.69)
 		)
 		(stroke
@@
 	(wire
 		(pts
+			(xy 170.18 67.31) (xy 187.96 67.31)
+		)
+		(stroke
+			(width 0)
+			(type default)
+		)
+	)
+	(wire
+		(pts
 			(xy 152.4 74.93) (xy 154.94 74.93)
 		)
@@
 		)
 	)
+	(wire
+		(pts
+			(xy 171.45 64.77) (xy 187.96 64.77)
+		)
+		(stroke
+			(width 0)
+			(type default)
+		)
+	)
 	(bus
 		(pts
@@
 		)
 	)
-	(wire
-		(pts
-			(xy 152.4 107.95) (xy 154.94 107.95)
-		)
-		(stroke
-			(width 0)
-			(type default)
-		)
-	)
 	(bus
 		(pts
@@
 	(wire
 		(pts
-			(xy 152.4 105.41) (xy 154.94 105.41)
-		)
-		(stroke
-			(width 0)
-			(type default)
-		)
-	)
-	(wire
-		(pts
 			(xy 15.24 25.4) (xy 15.24 22.86)
 		)
@@
 	(wire
 		(pts
+			(xy 152.4 143.51) (xy 154.94 143.51)
+		)
+		(stroke
+			(width 0)
+			(type default)
+		)
+	)
+	(wire
+		(pts
 			(xy 68.58 72.39) (xy 90.17 72.39)
 		)
@@
 	(wire
 		(pts
-			(xy 175.26 62.23) (xy 187.96 62.23)
+			(xy 170.18 62.23) (xy 187.96 62.23)
 		)
 		(stroke
@@
 		)
 	)
-	(label "BTN.1"
-		(at 154.94 95.25 0)
+	(label "MAX_SPI.SCK"
+		(at 154.94 143.51 0)
 		(fields_autoplaced yes)
 		(effects
@@
 		)
 	)
-	(label "MAX_SPI.SCK"
-		(at 154.94 107.95 0)
+	(label "BTN.1"
+		(at 154.94 95.25 0)
 		(fields_autoplaced yes)
 		(effects
@@
 		)
 	)
-	(label "MAX_SPI.RX"
-		(at 175.26 59.69 0)
+	(label "MAX_SPI.RX0"
+		(at 171.45 59.69 0)
 		(fields_autoplaced yes)
 		(effects
@@
 		)
 	)
-	(label "MAX_SPI.SCK"
-		(at 175.26 62.23 0)
+	(label "MAX_SPI.SCK1"
+		(at 170.18 62.23 0)
 		(fields_autoplaced yes)
 		(effects
@@
 		)
 	)
+	(label "MAX_SPI.RX"
+		(at 154.94 148.59 0)
+		(fields_autoplaced yes)
+		(effects
+			(font
+				(size 1.27 1.27)
+			)
+			(justify left bottom)
+		)
+	)
 	(label "SCREEN.SCL"
 		(at 175.26 93.98 0)
@@
 		)
 	)
+	(label "MAX_SPI.SCK[0..1]"
+		(at 170.18 67.31 0)
+		(fields_autoplaced yes)
+		(effects
+			(font
+				(size 1.27 1.27)
+			)
+			(justify left bottom)
+		)
+	)
 	(label "SDIO.CLK"
 		(at 184.15 100.33 180)
@@
 		)
 	)
+	(label "MAX_SPI.RX[0..1]"
+		(at 171.45 64.77 0)
+		(fields_autoplaced yes)
+		(effects
+			(font
+				(size 1.27 1.27)
+			)
+			(justify left bottom)
+		)
+	)
 	(label "DEBUG.SWCLK"
 		(at 33.02 147.32 0)
@@
 		)
 	)
-	(label "PI_TEMP_~{CS}.1"
+	(label "MAX_SPI_~{CS}1"
 		(at 196.85 67.31 0)
 		(fields_autoplaced yes)
@@
 		)
 	)
-	(label "MAX_SPI.RX"
-		(at 154.94 105.41 0)
-		(fields_autoplaced yes)
-		(effects
-			(font
-				(size 1.27 1.27)
-			)
-			(justify left bottom)
-		)
-	)
 	(label "FAN.1"
 		(at 186.69 49.53 180)
@@
 		)
 	)
-	(label "PI_TEMP_~{CS}.0"
+	(label "MAX_SPI.~{CS}0"
 		(at 196.85 64.77 0)
 		(fields_autoplaced yes)
@@
 		)
 	)
-	(hierarchical_label "BTN{0..2} SCREEN{SDA SCL} SPK"
-		(shape bidirectional)
-		(at 193.04 73.66 0)
-		(fields_autoplaced yes)
-		(effects
-			(font
-				(size 1.27 1.27)
-			)
-			(justify left)
-		)
-	)
-	(hierarchical_label "MAX_SPI{SCK RX} PI_TEMP_~{CS}[0..1] SSR[0..1] FAN[0..1]"
-		(shape bidirectional)
-		(at 193.04 45.72 0)
-		(fields_autoplaced yes)
-		(effects
-			(font
-				(size 1.27 1.27)
-			)
-			(justify left)
-		)
-	)
 	(hierarchical_label "~{RESET}"
 		(shape input)
@@
 		)
 	)
-	(hierarchical_label "SDIO{SMD CLK D[0..3]} ~{SD_DET}"
-		(shape bidirectional)
-		(at 191.77 96.52 0)
-		(fields_autoplaced yes)
-		(effects
-			(font
-				(size 1.27 1.27)
-			)
-			(justify left)
-		)
-	)
-	(hierarchical_label "QSPI{SD[0..3] SCLK CSN[0..1]}"
-		(shape bidirectional)
-		(at 71.12 107.95 180)
-		(fields_autoplaced yes)
-		(effects
-			(font
-				(size 1.27 1.27)
-			)
-			(justify right)
-		)
-	)
 	(symbol
 		(lib_id "power:GND")
@@
 			)
 		)
-		(property "Footprint" ""
+		(property "Footprint" "LED_SMD:LED_0805_2012Metric"
 			(at 25.4 58.42 90)
 			(effects
@@
 			)
 		)
-		(property "Footprint" ""
+		(property "Footprint" "Connector_JST:JST_XH_B3B-XH-AM_1x03_P2.50mm_Vertical"
 			(at 26.67 149.86 0)
 			(effects
@@
 			)
 		)
+		(pin "SDIO{SMD CLK D[0..3]} ~{SD_DET}" input
+			(at 191.77 96.52 180)
+			(effects
+				(font
+					(size 1.27 1.27)
+				)
+				(justify left)
+			)
+		)
 		(instances
 			(project "neflow"
@@
 			)
 		)
+		(pin "BTN{0..2} SCREEN{SDA SCL} SPK" bidirectional
+			(at 193.04 73.66 180)
+			(effects
+				(font
+					(size 1.27 1.27)
+				)
+				(justify left)
+			)
+		)
 		(instances
 			(project "neflow"
@@
 			)
 		)
+		(pin "QSPI{SD[0..3] SCLK CSN[0..1]}" bidirectional
+			(at 71.12 107.95 0)
+			(effects
+				(font
+					(size 1.27 1.27)
+				)
+				(justify right)
+			)
+		)
 		(instances
 			(project "neflow"
@@
 			)
 		)
+		(pin "MAX_SPI{SCK[0..1] RX[0..1] ~{CS}[0..1]} SSR[0..1] FAN[0..1]" bidirectional
+			(at 193.04 45.72 180)
+			(effects
+				(font
+					(size 1.27 1.27)
+				)
+				(justify left)
+			)
+		)
