File: pcb/temp_control.kicad_sch (KiCad schematic)
At the start: 30 parts, among them J501 Temp0, J502 Temp1, J503 SSR0, J504 SSR1, J505 FAN0, J506 FAN1, Q501 IRLML2502, Q502 IRLML2502, Q503 IRLML2502, Q504 IRLML2502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

Commit message: WIP: Stashing work to mess with vm
Connections:
- net PI_TEMP_~{CS}.0 renamed MAX_SPI.~{CS}0
- net PI_TEMP_~{CS}.1 renamed MAX_SPI.~{CS}1
Changed lines of the file:
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@@
-		)
-	)
-	(label "PI_TEMP_~{CS}.1"
-		(at 213.36 86.36 0)
-		(fields_autoplaced yes)
-		(effects
-			(font
-				(size 1.27 1.27)
-			)
-			(justify left bottom)
 		)
 	)
@@
 		)
 	)
-	(label "PI_TEMP_~{CS}.0"
-		(at 124.46 85.09 0)
-		(fields_autoplaced yes)
-		(effects
-			(font
-				(size 1.27 1.27)
-			)
-			(justify left bottom)
-		)
-	)
 	(label "MAX_SPI.RX"
 		(at 213.36 81.28 0)
@@
 		)
 	)
+	(label "MAX_SPI.RX"
+		(at 21.59 52.07 0)
+		(fields_autoplaced yes)
+		(effects
+			(font
+				(size 1.27 1.27)
+			)
+			(justify left bottom)
+		)
+	)
+	(label "FAN.1"
+		(at 21.59 59.69 0)
+		(fields_autoplaced yes)
+		(effects
+			(font
+				(size 1.27 1.27)
+			)
+			(justify left bottom)
+		)
+	)
+	(label "MAX_SPI.~{CS}0"
+		(at 124.46 85.09 0)
+		(fields_autoplaced yes)
+		(effects
+			(font
+				(size 1.27 1.27)
+			)
+			(justify left bottom)
+		)
+	)
+	(label "T1+"
+		(at 158.75 80.01 0)
+		(fields_autoplaced yes)
+		(effects
+			(font
+				(size 1.27 1.27)
+			)
+			(justify left bottom)
+		)
+	)
+	(label "MAX_SPI.SCK"
+		(at 21.59 49.53 0)
+		(fields_autoplaced yes)
+		(effects
+			(font
+				(size 1.27 1.27)
+			)
+			(justify left bottom)
+		)
+	)
+	(label "TC0+"
+		(at 81.28 78.74 0)
+		(fields_autoplaced yes)
+		(effects
+			(font
+				(size 1.27 1.27)
+			)
+			(justify left bottom)
+		)
+	)
+	(label "MAX_SPI.~{CS}0"
+		(at 24.13 45.72 0)
+		(fields_autoplaced yes)
+		(effects
+			(font
+				(size 1.27 1.27)
+			)
+			(justify left bottom)
+		)
+	)
+	(label "SSR.1"
+		(at 21.59 54.61 0)
+		(fields_autoplaced yes)
+		(effects
+			(font
+				(size 1.27 1.27)
+			)
+			(justify left bottom)
+		)
+	)
+	(label "SSR.1"
+		(at 195.58 127 0)
+		(fields_autoplaced yes)
+		(effects
+			(font
+				(size 1.27 1.27)
+			)
+			(justify left bottom)
+		)
+	)
+	(label "MAX_SPI.~{CS}1"
+		(at 213.36 86.36 0)
+		(fields_autoplaced yes)
+		(effects
+			(font
+				(size 1.27 1.27)
+			)
+			(justify left bottom)
+		)
+	)
+	(label "T0-"
+		(at 71.12 83.82 0)
+		(fields_autoplaced yes)
+		(effects
+			(font
+				(size 1.27 1.27)
+			)
+			(justify left bottom)
+		)
+	)
+	(label "MAX_SPI.SCK"
+		(at 213.36 78.74 0)
+		(fields_autoplaced yes)
+		(effects
+			(font
+				(size 1.27 1.27)
+			)
+			(justify left bottom)
+		)
+	)
 	(label "MAX_SPI.SCK"
 		(at 124.46 77.47 0)
@@
 		)
 	)
-	(label "MAX_SPI.RX"
-		(at 21.59 52.07 0)
-		(fields_autoplaced yes)
-		(effects
-			(font
-				(size 1.27 1.27)
-			)
-			(justify left bottom)
-		)
-	)
-	(label "FAN.1"
-		(at 21.59 59.69 0)
-		(fields_autoplaced yes)
-		(effects
-			(font
-				(size 1.27 1.27)
-			)
-			(justify left bottom)
-		)
-	)
-	(label "T1+"
-		(at 158.75 80.01 0)
-		(fields_autoplaced yes)
-		(effects
-			(font
-				(size 1.27 1.27)
-			)
-			(justify left bottom)
-		)
-	)
-	(label "MAX_SPI.SCK"
-		(at 21.59 49.53 0)
-		(fields_autoplaced yes)
-		(effects
-			(font
-				(size 1.27 1.27)
-			)
-			(justify left bottom)
-		)
-	)
-	(label "TC0+"
-		(at 81.28 78.74 0)
-		(fields_autoplaced yes)
-		(effects
-			(font
-				(size 1.27 1.27)
-			)
-			(justify left bottom)
-		)
-	)
-	(label "PI_TEMP_~{CS}.0"
-		(at 24.13 45.72 0)
-		(fields_autoplaced yes)
-		(effects
-			(font
-				(size 1.27 1.27)
-			)
-			(justify left bottom)
-		)
-	)
-	(label "SSR.1"
-		(at 21.59 54.61 0)
-		(fields_autoplaced yes)
-		(effects
-			(font
-				(size 1.27 1.27)
-			)
-			(justify left bottom)
-		)
-	)
-	(label "SSR.1"
-		(at 195.58 127 0)
-		(fields_autoplaced yes)
-		(effects
-			(font
-				(size 1.27 1.27)
-			)
-			(justify left bottom)
-		)
-	)
-	(label "T0-"
-		(at 71.12 83.82 0)
-		(fields_autoplaced yes)
-		(effects
-			(font
-				(size 1.27 1.27)
-			)
-			(justify left bottom)
-		)
-	)
-	(label "MAX_SPI.SCK"
-		(at 213.36 78.74 0)
-		(fields_autoplaced yes)
-		(effects
-			(font
-				(size 1.27 1.27)
-			)
-			(justify left bottom)
-		)
-	)
-	(label "PI_TEMP_~{CS}.1"
+	(label "MAX_SPI.~{CS}1"
 		(at 24.13 27.94 0)
 		(fields_autoplaced yes)
@@
 		)
 	)
-	(hierarchical_label "MAX_SPI{SCK RX} PI_TEMP_~{CS}[0..1] SSR[0..1] FAN[0..1]"
+	(hierarchical_label "MAX_SPI{SCK RX ~{CS}[0..1]} SSR[0..1] FAN[0..1]"
 		(shape bidirectional)
 		(at 19.05 66.04 0)
